File: kicad-project/anglerfish/anglerfish.kicad_pcb (KiCad board)
At the start: 2 copper layers, 276.9 x 188 mm, 73 parts, among them J1 Hirose_FH12-34S-0.5SH_1x34, U1 APDS-9306-065

Commit message: Generated gerbers. I discovered that I was working in a temp folder, so I erased the files under the anglerfish folder and manually brought the files from the temp folder.
Parts:
- added TP10: TestPoint, TestPoint:TestPoint_Pad_D1.5mm, B.Cu at (214.0, 53.0)
- added TP11: TestPoint, TestPoint:TestPoint_Pad_D1.5mm, B.Cu at (123.8, 124.1)
- added TP12: TestPoint, TestPoint:TestPoint_Pad_D1.5mm, B.Cu at (214.0, 58.0)
- added TP13: TestPoint, TestPoint:TestPoint_Pad_D1.5mm, B.Cu at (214.0, 62.0)
- added TP14: TestPoint, TestPoint:TestPoint_Pad_D1.5mm, B.Cu at (66.0, 51.5)
- added TP15: TestPoint, TestPoint:TestPoint_Pad_D1.5mm, B.Cu at (66.0, 59.2)
Connections:
- C2 pad 1: Net-(C2-Pad1) -> +5V
- D1 pad 1: Net-(C2-Pad1) -> +5V
- J1 pad 9: GND -> /photodiode-int
- TP3 pad 1: /photodiode-1/photodiode-int -> /photodiode-int
- U1 pad 4: /photodiode-1/photodiode-int -> /photodiode-int
Routing:
- net +5V: track 0.50 -> 190.1 mm, vias 0 -> 1
- net /photodiode-int: track 0.00 -> 121.1 mm, vias 0 -> 1
- net +3V3: track 114.9 -> 125.5 mm
- net GND: track 25.1 -> 18.3 mm, vias 9 -> 13
- net Net-(C2-Pad1): track 4.89 -> 0.00 mm, vias 1 -> 0
- net /led-apa102-1/apa102-cki: track 182.9 -> 186.8 mm
- net /led-apa102-1/apa102-sdi: track 182.2 -> 185.8 mm
- net /photodiode-1/photodiode-int: track 3.11 -> 0.00 mm, vias 1 -> 0
- net /LED_GROUP_1: track 180.6 -> 179.1 mm
- net /LED_GROUP_4: track 201.6 -> 200.6 mm
- net /photodiode-sda: track 115.0 -> 114.2 mm
- net /LED_GROUP_3: track 172.0 -> 172.8 mm
Other:
- board size 276.9 x 188 mm -> 281 x 221 mm
- board text added: "Iskender & Carina 2021"
- board text removed: "need to create a hole in fish's light to fit the digi led."
- board text removed: "these parts will look ugly. clean up."
